File: pathfinder.kicad_pcb (KiCad board)
At the start: 2 copper layers, 84.9 x 89.4 mm, 11 parts, among them SW1 SW_Push, SW2 SW_Push, SW3 SW_Push, SW4 SW_Push, U1 XIAO-RP2040-DIP

Commit message: Add files via upload
Parts:
- added D3: L08R5000Q1, footprints:LEDRD254W57D500H1070, F.Cu at (188.7, 97.4)
- added R3: R, Resistor_THT:R_Axial_DIN0204_L3.6mm_D1.6mm_P5.08mm_Horizontal, F.Cu at (213.6, 114.5)
- moved U1 1.53 mm to (188.7, 82.0)
Connections:
- U1 pad 3: unconnected-(U1-GPIO28/ADC2/A2-Pad3) -> LED3
Routing:
- net LED3: track 0.00 -> 45.6 mm
- net Net-(D3-PadA): track 0.00 -> 32.5 mm
- net GND: track 192.5 -> 223.8 mm
- net SW3: track 48.1 -> 52.8 mm
- net SW1: track 42.9 -> 45.1 mm
- net LED2: track 30.2 -> 31.1 mm
