File: pathfinder.kicad_sch (KiCad schematic)
At the start: 9 parts, among them SW1 SW_Push, SW2 SW_Push, SW3 SW_Push, SW4 SW_Push, U1 XIAO-RP2040-DIP

Commit message: Add files via upload
Parts:
- added D3: L08R5000Q1, footprints:LEDRD254W57D500H1070, symbol L08R5000Q1:L08R5000Q1
- added R3: R, Resistor_THT:R_Axial_DIN0204_L3.6mm_D1.6mm_P5.08mm_Horizontal, symbol Device:R
Connections:
- net GND: now also D3.C
- net LED3: now reaches U1.3 (GPIO28/ADC2/A2)
- net LED3: now also R3.2
- new net: D3.A, R3.1
